Commit message: feat(gui): пульт робота — карта (pan/zoom) + камера + кастомизация, дизайн ZMK Vision
- gui/: React 19 + Vite 6 + TS, дизайн-система перенесена из
  danilka-revin/zmk-videoanalytics (токены, тёмная/светлая темы,
  лаймовый акцент, сайдбар, панели, сегментный тумблер)
- тумблер «Карта / Камера» по центру шапки (клавиши 1/2, K — настройки)
- карта SLAM на canvas: сдвиг ЛКМ/пинч, зум колесом к курсору,
  кнопки +/−/вписать/следование за роботом, сетка в метрах,
  масштабная линейка, компас, шлейф, облако точек скана, цель
- робот 0.75×0.60 м с 4 модулями; лидар ЛДС-01 — сверху спереди по
  центру (URDF lidar_joint x=0.32), вращающийся луч скана
- окно камеры: демо-рейкастинг от позиции робота (реагирует на
  движение/поворот), LIVE/DEMO-бейдж, HUD, сетка, снимок PNG,
  fullscreen; при URL потока — <video>
- кастомизация: тема (светлая/тёмная/авто), акцент (5 пресетов),
  шрифт S/M/L, стиль карты, следование, сетка/шлейф/скан, масштаб
  метки, качество камеры, оверлеи, URL потока, сброс; всё в localStorage
- демо-симулятор 10 Гц: крабовая кинематика, 360° DDA-скан из носовой
  точки, батарея/одометр; источник данных изолирован под мост ROS 2
- URDF: лидар передвинут на переднюю центральную верхнюю точку
- README: строка навигации на gui/

Co-authored-by: arena-agent <297053741+arena-agent@users.noreply.github.com>

File: ros2_ws/src/rus_slam_description/urdf/rus_slam.urdf.xacro (robot description, xacro)
@@ -99,5 +99,5 @@
   <xacro:swerve_module prefix="rr" x="${-wheelbase/2}" y="${-track/2}"/>
   <!-- ============================== сенсоры ============================= -->
-  <!-- Лидар ЛДС-01: на верхней палубе, ближе к носу -->
+  <!-- Лидар ЛДС-01: на верхней палубе, спереди по центру (x = 0.32 м от center) -->
   <link name="lidar_link">
     <visual>
@@ -117,5 +117,5 @@
     <parent link="base_link"/>
     <child link="lidar_link"/>
-    <origin xyz="0.25 0 0.32" rpy="0 0 0"/>
+    <origin xyz="0.32 0 0.32" rpy="0 0 0"/>
   </joint>
   <!-- Камера машинного зрения -->
